Commit message: Update inertia

File: omnibot_description/urdf/base.urdf.xacro (robot description, xacro)
@@ -5,9 +5,9 @@
       <inertial>
         <origin xyz="0.0 0.0 0.0" rpy="0.0 0.0 0.0"/>
-        <mass value="0.325"/>
-        <inertia ixx="0.00112318" ixy="-4.044e-6" ixz="-1.882e-6" iyy="0.002" iyz="9.405e-7" izz="0.003"/>
+        <mass value="2.067"/>
+        <inertia ixx="0.00465053" ixy="1.014e-6" ixz="-1.413e-5" iyy="0.00771714" iyz="2.949e-6" izz="0.01114849"/>
       </inertial>
       <visual>
-        <origin xyz="0.0 0.0 0.0" rpy="0.0 0.0 0.0"/>
+        <origin xyz="0.0 0.0 -0.013" rpy="0.0 0.0 0.0"/>
         <geometry>
           <!-- <box size="${base_length} ${base_width} ${base_height}"/> -->

File: omnibot_description/urdf/sensors.urdf.xacro (robot description, xacro)
@@ -26,7 +26,7 @@
       </collision>
       <inertial>
-        <origin xyz="0 0 0" rpy="0 0 0"/>
-        <mass value="0.125"/>
-        <inertia ixx="0.001"  ixy="0"  ixz="0" iyy="0.001" iyz="0" izz="0.001" />
+        <origin xyz="0.009 0 0.01" rpy="0 0 0"/>
+        <mass value="0.165"/>
+        <inertia ixx="6.790e-5" ixy="2.124e-5" ixz="0" iyy="1.305e-4" iyz="0" izz="1.572e-4" />
       </inertial>
     </link>

File: omnibot_description/urdf/wheel.urdf.xacro (robot description, xacro)
@@ -18,6 +18,6 @@
       <inertial>
         <origin xyz="0.0 0.0 0.0" rpy="0.0 0.0 0.0"/>
-        <mass value="0.060"/>
-        <inertia ixx="1e-6" ixy="0.0" ixz="0.0" iyy="1e-6" iyz="0.0" izz="1e-6"/>
+        <mass value="0.120"/>
+        <inertia ixx="6.278e-5" ixy="2.396e-10" ixz="4.709e-11" iyy="9.349e-5" iyz="-1.916e-10" izz="6.278e-5"/>
       </inertial>
     </link>

Commit message: Add Lidar plugin

File: omnibot_description/urdf/base.urdf.xacro (robot description, xacro)
@@ -4,13 +4,14 @@
     <link name="base_link">
       <inertial>
-        <origin xyz="0.0 0.0 0.0" rpy="0.0 0.0 0.0"/>
+        <origin xyz="0.0 0.0 -0.013" rpy="0.0 0.0 0.0"/>
         <mass value="2.067"/>
         <inertia ixx="0.00465053" ixy="1.014e-6" ixz="-1.413e-5" iyy="0.00771714" iyz="2.949e-6" izz="0.01114849"/>
       </inertial>
       <visual>
-        <origin xyz="0.0 0.0 -0.013" rpy="0.0 0.0 0.0"/>
+        <origin xyz="0.0 0.0 0.0" rpy="0.0 0.0 0.0"/>
         <geometry>
           <!-- <box size="${base_length} ${base_width} ${base_height}"/> -->
-          <mesh filename="package://omnibot_description/meshes/base_link.dae"/>
+          <!-- <mesh filename="package://omnibot_description/meshes/base_link.dae"/> -->
+          <mesh filename="$(find omnibot_description)/meshes/base_link.dae"/>
         </geometry>
       </visual>

File: omnibot_description/urdf/omnibot.urdf.xacro (robot description, xacro)
@@ -30,5 +30,5 @@
   </xacro:imu>
   <xacro:lidar>
-    <origin xyz="-0.013 0.0 ${base_height/2 + 0.01}" rpy="0.0 0.0 0.0"/>
+    <origin xyz="-0.013 0.0 ${base_height/2 + 0.024}" rpy="0.0 0.0 0.0"/>
   </xacro:lidar>
   <xacro:camera>

File: omnibot_description/urdf/sensors.urdf.xacro (robot description, xacro)
@@ -14,17 +14,20 @@
     <link name="lidar_link">
       <visual>
-        <origin xyz="0 0 0" rpy="0 0 0"/>
+        <origin xyz="0 0 -0.014" rpy="0 0 0"/>
         <geometry>
-          <mesh filename="package://omnibot_description/meshes/lidar.dae"/>
+          <!-- <mesh filename="package://omnibot_description/meshes/lidar.dae"/> -->
+          <mesh filename="$(find omnibot_description)/meshes/lidar.dae"/>
         </geometry>
       </visual>
       <collision>
-        <origin xyz="0 0 0" rpy="0 0 0"/>
+        <origin xyz="0 0 -0.014" rpy="0 0 0"/>
         <geometry>
-          <cylinder radius="0.0508" length="0.04"/>
+          <!-- <cylinder radius="0.0508" length="0.04"/> -->
+          <!-- <mesh filename="package://omnibot_description/meshes/lidar.stl"/> -->
+          <mesh filename="$(find omnibot_description)/meshes/lidar.stl"/>
         </geometry>
       </collision>
       <inertial>
-        <origin xyz="0.009 0 0.01" rpy="0 0 0"/>
+        <origin xyz="0.009 0 -0.04" rpy="0 0 0"/>
         <mass value="0.165"/>
         <inertia ixx="6.790e-5" ixy="2.124e-5" ixz="0" iyy="1.305e-4" iyz="0" izz="1.572e-4" />
@@ -36,4 +39,38 @@
       <xacro:insert_block name="joint_pose"/>
     </joint>
+    <gazebo reference="lidar_link">
+      <sensor name='gpu_lidar' type='gpu_lidar'>"
+        <topic>lidar</topic>
+        <update_rate>30</update_rate>
+        <ray>
+          <scan>
+            <horizontal>
+              <samples>720</samples>
+              <resolution>1</resolution>
+              <min_angle>-3.1415</min_angle>
+              <max_angle>3.1415</max_angle>
+            </horizontal>
+            <vertical>
+              <samples>1</samples>
+              <resolution>0.01</resolution>
+              <min_angle>0</min_angle>
+              <max_angle>0</max_angle>
+            </vertical>
+          </scan>
+          <range>
+            <min>0.05</min>
+            <max>8.0</max>
+            <resolution>0.01</resolution>
+          </range>
+          <noise>
+            <type>gaussian</type>
+            <mean>0.0</mean>
+            <stddev>0.01</stddev>
+          </noise>
+        </ray>
+        <always_on>1</always_on>
+        <visualize>true</visualize>
+      </sensor>
+    </gazebo>
   </xacro:macro>
   <!-- Camera macro -->
@@ -48,5 +85,6 @@
         <origin xyz="0.0 0.0 0.0" rpy="0.0 0.0 0.0"/>
         <geometry>
-          <mesh filename="package://omnibot_description/meshes/raspicam.dae"/>
+          <!-- <mesh filename="package://omnibot_description/meshes/raspicam.dae"/> -->
+          <mesh filename="$(find omnibot_description)/meshes/raspicam.dae"/>
         </geometry>
       </visual>

File: omnibot_description/urdf/wheel.urdf.xacro (robot description, xacro)
@@ -6,6 +6,7 @@
         <origin xyz="0.0 0.0 0.0" rpy="0.0 0.0 0.0"/>
         <geometry>
-          <mesh filename="package://omnibot_description/meshes/mecanum_wheel_${prefix}.dae"/>
           <!-- <cylinder radius="${wheel_radius}" length="${wheel_width}"/> -->
+          <!-- <mesh filename="package://omnibot_description/meshes/mecanum_wheel_${prefix}.dae"/> -->
+          <mesh filename="$(find omnibot_description)/meshes/mecanum_wheel_${prefix}.dae"/>
         </geometry>
       </visual>
