Commit message: Fix urdf

File: omnibot_description/urdf/omnibot.urdf.xacro (robot description, xacro)
@@ -1,20 +1,20 @@
 <?xml version="1.0"?>
 <robot xmlns:xacro="http://www.ros.org/wiki/xacro" name="omnibot">
-  <xacro:property name="base_length" value="0.30"/>
-  <xacro:property name="base_width" value="0.20"/>
-  <xacro:property name="base_height" value="0.10"/>
-  <xacro:property name="wheel_length" value="0.030"/>
+  <xacro:property name="base_length" value="0.28"/>
+  <xacro:property name="base_width" value="0.18"/>
+  <xacro:property name="base_height" value="0.08"/>
+  <xacro:property name="wheel_width" value="0.030"/>
   <xacro:property name="wheel_radius" value="0.032"/>
   <xacro:property name="wheel_x_offset" value="${base_length/4}"/>
-  <xacro:property name="wheel_y_offset" value="${base_widht/2 + 0.01}"/>
+  <xacro:property name="wheel_y_offset" value="${base_width/2 + wheel_width/2 + 0.005}"/>
   <xacro:property name="wheel_z_offset" value="${-base_height/2 + 0.02}"/>
-  <xacro:property name="PI" value="3.14159"/>
+  <xacro:property name="M_PI" value="3.14159"/>
   <xacro:macro name="omnibot_wheel" params="prefix *joint_pose">
     <link name="${prefix}_wheel_link">
       <visual>
-        <origin xyz="0.0 0.0 0.0" rpy="0.0 0.0 0.0"/>
+        <origin xyz="0.0 0.0 0.0" rpy="${M_PI/2} 0.0 0.0"/>
         <geometry>
           <!-- <mesh filename="package://omnibot_description/meshes/omni_wheel.dae"/> -->
-          <cylinder radius="${wheel_radius}" length="${wheel_length}"/>
+          <cylinder radius="${wheel_radius}" length="${wheel_width}"/>
         </geometry>
         <material name="LightGrey">
@@ -23,8 +23,8 @@
       </visual>
       <collision>
-        <origin xyz="0.0 0.0 0.0" rpy="0.0 0.0 0.0"/>
+        <origin xyz="0.0 0.0 0.0" rpy="${M_PI/2} 0.0 0.0"/>
         <geometry>
           <!-- <mesh filename="package://omnibot_description/meshes/omni_wheel.stl"/> -->
-          <cylinder radius="${wheel_radius}" length="${wheel_length}"/>
+          <cylinder radius="${wheel_radius}" length="${wheel_width}"/>
         </geometry>
       </collision>
@@ -69,5 +69,5 @@
     <parent link="base_link"/>
     <child link="base_footprint"/>
-    <origin xyz="0.0 0.0 ${-(wheel_radius+wheel_z_offset)}" rpy="0 0 0"/>
+    <origin xyz="0.0 0.0 ${-(wheel_radius-wheel_z_offset)}" rpy="0 0 0"/>
   </joint>
   <xacro:omnibot_wheel prefix="front_left">

Commit message: Add sensors and spawn gazebo

File: omnibot_description/urdf/omnibot.urdf.xacro (robot description, xacro)
@@ -10,4 +10,5 @@
   <xacro:property name="wheel_z_offset" value="${-base_height/2 + 0.02}"/>
   <xacro:property name="M_PI" value="3.14159"/>
+  <xacro:include filename="$(find omnibot_description)/urdf/sensors.urdf.xacro"/>
   <xacro:macro name="omnibot_wheel" params="prefix *joint_pose">
     <link name="${prefix}_wheel_link">
@@ -31,5 +32,5 @@
       <inertial>
         <origin xyz="0.0 0.0 0.0" rpy="0.0 0.0 0.0"/>
-        <mass value="0.050"/>
+        <mass value="0.060"/>
         <inertia ixx="1e-6" ixy="0.0" ixz="0.0" iyy="1e-6" iyz="0.0" izz="1e-6"/>
       </inertial>
@@ -45,6 +46,6 @@
     <inertial>
       <origin xyz="0.0 0.0 0.0" rpy="0.0 0.0 0.0"/>
-      <mass value="1.0"/>
-      <inertia ixx="1e-6" ixy="0.0" ixz="0.0" iyy="1e-6" iyz="0.0" izz="1e-6"/>
+      <mass value="3.0"/>
+      <inertia ixx="1e-4" ixy="0.0" ixz="0.0" iyy="1e-4" iyz="0.0" izz="1e-4"/>
     </inertial>
     <visual name="">
@@ -83,3 +84,12 @@
     <origin xyz="${-wheel_x_offset} ${wheel_y_offset} ${wheel_z_offset}" rpy="0.0 0.0 0.0"/>
   </xacro:omnibot_wheel>
+  <xacro:imu>
+    <origin xyz="0.0 0.0 0.0" rpy="0.0 0.0 0.0"/>
+  </xacro:imu>
+  <xacro:lidar>
+    <origin xyz="0.0 0.0 ${base_height/2 + 0.02}" rpy="0.0 0.0 0.0"/>
+  </xacro:lidar>
+  <xacro:camera>
+    <origin xyz="${base_length/2} 0.0 ${base_height/2}" rpy="0.0 0.0 0.0"/>
+  </xacro:camera>
 </robot>

Commit message: Update inertia base_link

File: omnibot_description/urdf/omnibot.urdf.xacro (robot description, xacro)
@@ -1,12 +1,12 @@
 <?xml version="1.0"?>
 <robot xmlns:xacro="http://www.ros.org/wiki/xacro" name="omnibot">
-  <xacro:property name="base_length" value="0.28"/>
-  <xacro:property name="base_width" value="0.18"/>
-  <xacro:property name="base_height" value="0.08"/>
-  <xacro:property name="wheel_width" value="0.030"/>
-  <xacro:property name="wheel_radius" value="0.032"/>
-  <xacro:property name="wheel_x_offset" value="${base_length/4}"/>
-  <xacro:property name="wheel_y_offset" value="${base_width/2 + wheel_width/2 + 0.005}"/>
-  <xacro:property name="wheel_z_offset" value="${-base_height/2 + 0.02}"/>
+  <xacro:property name="base_length" value="0.200"/>
+  <xacro:property name="base_width" value="0.140"/>
+  <xacro:property name="base_height" value="0.0764"/>
+  <xacro:property name="wheel_width" value="0.036"/>
+  <xacro:property name="wheel_radius" value="0.039"/>
+  <xacro:property name="wheel_x_offset" value="0.06"/>
+  <xacro:property name="wheel_y_offset" value="${base_width/2 + wheel_width/2 + 0.0165}"/>
+  <xacro:property name="wheel_z_offset" value="${-base_height/2 + 0.0228}"/>
   <xacro:property name="M_PI" value="3.14159"/>
   <xacro:macro name="omnibot_wheel" params="prefix *joint_pose">
@@ -45,16 +45,13 @@
     <inertial>
       <origin xyz="0.0 0.0 0.0" rpy="0.0 0.0 0.0"/>
-      <mass value="1.0"/>
-      <inertia ixx="1e-6" ixy="0.0" ixz="0.0" iyy="1e-6" iyz="0.0" izz="1e-6"/>
+      <mass value="0.325"/>
+      <inertia ixx="0.00112318" ixy="-4.044e-6" ixz="-1.882e-6" iyy="0.002" iyz="9.405e-7" izz="0.003"/>
     </inertial>
-    <visual name="">
+    <visual>
       <origin xyz="0.0 0.0 0.0" rpy="0.0 0.0 0.0"/>
       <geometry>
         <box size="${base_length} ${base_width} ${base_height}"/>
+        <!-- <mesh filename="package://omnibot_description/meshes/base_link.stl"/> -->
       </geometry>
-      <material name="">
-        <color rgba="1.0 0.0 0.0 1.0"/>
-        <!-- <texture filename=""/> -->
-      </material>
     </visual>
     <collision>
@@ -83,3 +80,12 @@
     <origin xyz="${-wheel_x_offset} ${wheel_y_offset} ${wheel_z_offset}" rpy="0.0 0.0 0.0"/>
   </xacro:omnibot_wheel>
+  <!-- <xacro:imu>
+    <origin xyz="0.0 0.0 0.0" rpy="0.0 0.0 0.0"/>
+  </xacro:imu>
+  <xacro:lidar>
+    <origin xyz="0.0 0.0 ${base_height/2 + 0.02}" rpy="0.0 0.0 0.0"/>
+  </xacro:lidar> -->
+  <!-- <xacro:camera>
+    <origin xyz="${base_length/2} 0.0 ${base_height/2}" rpy="0.0 0.0 0.0"/>
+  </xacro:camera> -->
 </robot>

Commit message: Create omni_world.sdf

File: omnibot_description/urdf/omnibot.urdf.xacro (robot description, xacro)
@@ -87,10 +87,9 @@
     <origin xyz="0.0 0.0 ${base_height/2 + 0.02}" rpy="0.0 0.0 0.0"/>
   </xacro:lidar>
-  <!-- <xacro:camera>
+  <xacro:camera>
     <origin xyz="${base_length/2} 0.0 ${base_height/2}" rpy="0.0 0.0 0.0"/>
-  </xacro:camera> -->
+  </xacro:camera>
   <gazebo>
-    <!-- Joint states plugin -->
-    <plugin filename="libignition-gazebo-joint-state-publisher-system.so"
+      <plugin filename="libignition-gazebo-joint-state-publisher-system.so"
             name="ignition::gazebo::systems::JointStatePublisher"/>
   </gazebo>

File: omnibot_description/urdf/sensors.urdf.xacro (robot description, xacro)
@@ -10,5 +10,5 @@
     </joint>
     <!-- IMU Plugin -->
-    <gazebo reference="imu_link">
+    <!-- <gazebo reference="imu_link">
       <sensor name="imu_sensor" type="imu">
         <plugin filename="ignition-gazebo-imu-system"
@@ -19,5 +19,5 @@
         <topic>imu</topic>
       </sensor>
-    </gazebo>
+    </gazebo> -->
   </xacro:macro>
   <!-- Lidar Plugin macro -->
@@ -48,33 +48,4 @@
     </joint>
     <!-- Lidar Plugin -->
-    <gazebo reference="lidar_link">
-      <sensor name='gpu_lidar' type='gpu_lidar'>"
-        <topic>scan</topic>
-        <update_rate>30</update_rate>
-        <ray>
-        <scan>
-            <horizontal>
-            <samples>640</samples>
-            <resolution>1</resolution>
-            <min_angle>-1.396263</min_angle>
-            <max_angle>1.396263</max_angle>
-            </horizontal>
-            <vertical>
-            <samples>1</samples>
-            <resolution>0.01</resolution>
-            <min_angle>0</min_angle>
-            <max_angle>0</max_angle>
-            </vertical>
-        </scan>
-        <range>
-            <min>0.08</min>
-            <max>10.0</max>
-            <resolution>0.01</resolution>
-        </range>
-        </ray>
-        <alwaysOn>1</alwaysOn>
-        <visualize>true</visualize>
-      </sensor>
-    </gazebo>
   </xacro:macro>
   <!-- Camera Plugin macro -->
@@ -92,4 +63,10 @@
         </geometry>
       </visual>
+      <collision>
+        <origin xyz="0.0 0.0 0.0" rpy="0.0 0.0 0.0"/>
+        <geometry>
+          <box size="0.001 0.025 0.024"/>
+        </geometry>
+      </collision>
     </link>
     <joint name="camera_joint" type="fixed">

Commit message: Update urdf meshes

File: omnibot_description/urdf/omnibot.urdf.xacro (robot description, xacro)
@@ -10,74 +10,19 @@
   <xacro:property name="wheel_z_offset" value="${-base_height/2 + 0.0228}"/>
   <xacro:property name="M_PI" value="3.14159"/>
+  <xacro:include filename="$(find omnibot_description)/urdf/base.urdf.xacro"/>
+  <xacro:include filename="$(find omnibot_description)/urdf/wheel.urdf.xacro"/>
   <xacro:include filename="$(find omnibot_description)/urdf/sensors.urdf.xacro"/>
-  <xacro:macro name="omnibot_wheel" params="prefix *joint_pose">
-    <link name="${prefix}_wheel_link">
-      <visual>
-        <origin xyz="0.0 0.0 0.0" rpy="${M_PI/2} 0.0 0.0"/>
-        <geometry>
-          <!-- <mesh filename="package://omnibot_description/meshes/omni_wheel.dae"/> -->
-          <cylinder radius="${wheel_radius}" length="${wheel_width}"/>
-        </geometry>
-        <material name="LightGrey">
-          <color rgba="0.7 0.7 0.7 1.0"/>
-        </material>
-      </visual>
-      <collision>
-        <origin xyz="0.0 0.0 0.0" rpy="${M_PI/2} 0.0 0.0"/>
-        <geometry>
-          <!-- <mesh filename="package://omnibot_description/meshes/omni_wheel.stl"/> -->
-          <cylinder radius="${wheel_radius}" length="${wheel_width}"/>
-        </geometry>
-      </collision>
-      <inertial>
-        <origin xyz="0.0 0.0 0.0" rpy="0.0 0.0 0.0"/>
-        <mass value="0.060"/>
-        <inertia ixx="1e-6" ixy="0.0" ixz="0.0" iyy="1e-6" iyz="0.0" izz="1e-6"/>
-      </inertial>
-    </link>
-    <joint name="${prefix}_wheel_joint" type="continuous">
-      <xacro:insert_block name="joint_pose"/>
-      <parent link="base_link"/>
-      <child link="${prefix}_wheel_link"/>
-      <axis xyz="0 1 0" rpy="0.0 0.0 0.0"/>
-    </joint>
-  </xacro:macro>
-  <link name="base_link">
-    <inertial>
-      <origin xyz="0.0 0.0 0.0" rpy="0.0 0.0 0.0"/>
-      <mass value="0.325"/>
-      <inertia ixx="0.00112318" ixy="-4.044e-6" ixz="-1.882e-6" iyy="0.002" iyz="9.405e-7" izz="0.003"/>
-    </inertial>
-    <visual>
-      <origin xyz="0.0 0.0 0.0" rpy="0.0 0.0 0.0"/>
-      <geometry>
-        <box size="${base_length} ${base_width} ${base_height}"/>
-        <!-- <mesh filename="package://omnibot_description/meshes/base_link.stl"/> -->
-      </geometry>
-    </visual>
-    <collision>
-      <origin xyz="0.0 0.0 0.0" rpy="0.0 0.0 0.0"/>
-      <geometry>
-        <box size="${base_length} ${base_width} ${base_height}"/>
-      </geometry>
-    </collision>
-  </link>
-  <link name="base_footprint"/>
-  <joint name="base_joint" type="fixed">
-    <parent link="base_link"/>
-    <child link="base_footprint"/>
-    <origin xyz="0.0 0.0 ${-(wheel_radius-wheel_z_offset)}" rpy="0 0 0"/>
-  </joint>
-  <xacro:omnibot_wheel prefix="front_left">
+  <xacro:omnibot_base/>
+  <xacro:omnibot_wheel prefix="front_right">
     <origin xyz="${wheel_x_offset} ${-wheel_y_offset} ${wheel_z_offset}" rpy="0.0 0.0 0.0"/>
   </xacro:omnibot_wheel>
-  <xacro:omnibot_wheel prefix="front_right">
+  <xacro:omnibot_wheel prefix="front_left">
     <origin xyz="${wheel_x_offset} ${wheel_y_offset} ${wheel_z_offset}" rpy="0.0 0.0 0.0"/>
   </xacro:omnibot_wheel>
   <xacro:omnibot_wheel prefix="back_left">
-    <origin xyz="${-wheel_x_offset} ${-wheel_y_offset} ${wheel_z_offset}" rpy="0.0 0.0 0.0"/>
+    <origin xyz="${-wheel_x_offset} ${wheel_y_offset} ${wheel_z_offset}" rpy="0.0 0.0 0.0"/>
   </xacro:omnibot_wheel>
   <xacro:omnibot_wheel prefix="back_right">
-    <origin xyz="${-wheel_x_offset} ${wheel_y_offset} ${wheel_z_offset}" rpy="0.0 0.0 0.0"/>
+    <origin xyz="${-wheel_x_offset} ${-wheel_y_offset} ${wheel_z_offset}" rpy="0.0 0.0 0.0"/>
   </xacro:omnibot_wheel>
   <xacro:imu>
@@ -85,8 +30,8 @@
   </xacro:imu>
   <xacro:lidar>
-    <origin xyz="0.0 0.0 ${base_height/2 + 0.02}" rpy="0.0 0.0 0.0"/>
+    <origin xyz="-0.013 0.0 ${base_height/2 + 0.01}" rpy="0.0 0.0 0.0"/>
   </xacro:lidar>
   <xacro:camera>
-    <origin xyz="${base_length/2} 0.0 ${base_height/2}" rpy="0.0 0.0 0.0"/>
+    <origin xyz="${base_length/2 - 0.0014} 0.0 0.018" rpy="0.0 0.0 0.0"/>
   </xacro:camera>
   <gazebo>

File: omnibot_description/urdf/sensors.urdf.xacro (robot description, xacro)
@@ -9,17 +9,6 @@
       <xacro:insert_block name="joint_pose"/>
     </joint>
-    <!-- IMU Plugin -->
-    <!-- <gazebo reference="imu_link">
-      <sensor name="imu_sensor" type="imu">
-        <plugin filename="ignition-gazebo-imu-system"
-                name="ignition::gazebo::systems::Imu"/>
-        <always_on>1</always_on>
-        <update_rate>30</update_rate>
-        <visualize>true</visualize>
-        <topic>imu</topic>
-      </sensor>
-    </gazebo> -->
   </xacro:macro>
-  <!-- Lidar Plugin macro -->
+  <!-- Lidar macro -->
   <xacro:macro name="lidar" params="*joint_pose">
     <link name="lidar_link">
@@ -27,5 +16,5 @@
         <origin xyz="0 0 0" rpy="0 0 0"/>
         <geometry>
-          <cylinder radius="0.0508" length="0.04"/>
+          <mesh filename="package://omnibot_description/meshes/lidar.dae"/>
         </geometry>
       </visual>
@@ -47,7 +36,6 @@
       <xacro:insert_block name="joint_pose"/>
     </joint>
-    <!-- Lidar Plugin -->
   </xacro:macro>
-  <!-- Camera Plugin macro -->
+  <!-- Camera macro -->
   <xacro:macro name="camera" params="*joint_pose">
     <link name="camera_link">
@@ -60,5 +48,5 @@
         <origin xyz="0.0 0.0 0.0" rpy="0.0 0.0 0.0"/>
         <geometry>
-          <box size="0.001 0.025 0.024"/>
+          <mesh filename="package://omnibot_description/meshes/raspicam.dae"/>
         </geometry>
       </visual>
@@ -75,5 +63,4 @@
       <xacro:insert_block name="joint_pose"/>
     </joint>
-    <!-- Camera Plugin -->
   </xacro:macro>
 </robot>

Commit message: Implement PreUpdate

File: omnibot_description/urdf/omnibot.urdf.xacro (robot description, xacro)
@@ -14,9 +14,9 @@
   <xacro:include filename="$(find omnibot_description)/urdf/sensors.urdf.xacro"/>
   <xacro:omnibot_base/>
+  <xacro:omnibot_wheel prefix="front_left">
+    <origin xyz="${wheel_x_offset} ${wheel_y_offset} ${wheel_z_offset}" rpy="0.0 0.0 0.0"/>
+  </xacro:omnibot_wheel>
   <xacro:omnibot_wheel prefix="front_right">
     <origin xyz="${wheel_x_offset} ${-wheel_y_offset} ${wheel_z_offset}" rpy="0.0 0.0 0.0"/>
-  </xacro:omnibot_wheel>
-  <xacro:omnibot_wheel prefix="front_left">
-    <origin xyz="${wheel_x_offset} ${wheel_y_offset} ${wheel_z_offset}" rpy="0.0 0.0 0.0"/>
   </xacro:omnibot_wheel>
   <xacro:omnibot_wheel prefix="back_left">
@@ -38,16 +38,4 @@
     <plugin filename="libignition-gazebo-joint-state-publisher-system.so"
             name="ignition::gazebo::systems::JointStatePublisher"/>
-    <!-- <plugin
-      filename="libignition-gazebo-diff-drive-system.so"
-      name="ignition::gazebo::systems::DiffDrive">
-      <left_joint>front_left_wheel_joint</left_joint>
-      <left_joint>back_left_wheel_joint</left_joint>
-      <right_joint>front_right_wheel_joint</right_joint>
-      <right_joint>back_right_wheel_joint</right_joint>
-      <wheel_separation>0.21</wheel_separation>
-      <wheel_radius>0.039</wheel_radius>
-      <topic>cmd_vel</topic>
-      <odom_topic>odom</odom_topic>
-    </plugin> -->
     <plugin
       filename="libOmniDrive.so"
